File: Kicad files/usb_c_pd_source.kicad_sch (KiCad schematic)
At the start: 53 parts, among them J1 Barrel_Jack, J2 Lab_supply, J3 Serial Wire, J4 USB4151-GF-C, Q1 DMP3013SFV-7, Q2 DMP3013SFV-7, Q3 DMP3013SFV-7, U1 TPS560430X3FDBVR, U2 TPS56837HRPAR, U3 STM32G030F6Px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

Commit message: Add files via upload
Parts:
- removed J1: Barrel_Jack, footprints:PJ106AHTR, symbol Connector:Barrel_Jack
- removed NT1: NetTie_2, NetTie:NetTie-2_SMD_Pad0.5mm, symbol Device:NetTie_2
- added NT2: NetTie_2, NetTie:NetTie-2_SMD_Pad0.5mm, symbol Device:NetTie_2
- C5, C8: footprint Capacitor_SMD:C_0805_2012Metric_Pad1.18x1.45mm_HandSolder -> Capacitor_SMD:C_0603_1608Metric
- C9: value 10u -> 4u7
- L1: value 12u -> 6u8; footprint footprints:SRR0735A120M -> Inductor_SMD:L_1008_2520Metric
- L2: footprint footprints:INDPM112100X400N -> Inductor_SMD:L_Taiyo-Yuden_MD-5050
- R1, R10, R11, R4, R6, R7, R8, R9: footprint Resistor_SMD:R_0805_2012Metric_Pad1.20x1.40mm_HandSolder -> Resistor_SMD:R_0603_1608Metric
- U1: value TPS560430X3FDBVR -> TPS560430YFDBVR
Connections:
- net AGND: now also NT2.1
- net GND: now also NT2.2
Other:
- note removed: "naj bo pozicioniran tako, da lahko priklopiš kar PCB na napravo"
- note removed: "obvezno preveri če je to tvoje napajanje!!!"
- note removed: "preveri če dela nucleo"
- note removed: "če boš v prihodnosti hotel krmiliti vklop z MCU"
- moved on the sheet: J2
